File: pcb/OPA846.kicad_sch (KiCad schematic)
At the start: 11 parts, among them J1 Conn_Coaxial, U1 OPA846

Commit message: updated readme a bit
Parts:
- C32: renamed from C27; value 47n -> 0u1
- renumbered C24 to C29, C25 to C30, C26 to C31, C28 to C33, J1 to J2, R6 to R10, R7 to R11, R8 to R12, R9 to R13, U1 to U2
Changed lines of the file:
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@@
 (kicad_sch (version 20200618) (host eeschema "(5.99.0-2251-g5226d6b4d)")
-  (page 2 9)
+  (page 3 9)
   (paper "User" 148.006 105.004)
   (title_block
@@
   (symbol (lib_name "nets:+5V-A_1") (lib_id "nets:+5V-A") (at 68.58 21.59 0)
     (in_bom yes) (on_board yes)
-    (property "Reference" "#PWR0123" (id 0) (at 68.58 25.4 0)
+    (property "Reference" "#PWR0125" (id 0) (at 68.58 25.4 0)
       (effects (font (size 1.27 1.27)) hide)
     )
@@
   (symbol (lib_id "nets:-5V") (at 68.58 40.64 180)
     (in_bom yes) (on_board yes)
-    (property "Reference" "#PWR054" (id 0) (at 68.58 43.18 0)
+    (property "Reference" "#PWR062" (id 0) (at 68.58 43.18 0)
       (effects (font (size 1.27 1.27)) hide)
     )
@@
   (symbol (lib_id "nets:+5V-A") (at 123.19 21.59 0)
     (in_bom yes) (on_board yes)
-    (property "Reference" "#PWR0124" (id 0) (at 123.19 25.4 0)
+    (property "Reference" "#PWR0126" (id 0) (at 123.19 25.4 0)
       (effects (font (size 1.27 1.27)) hide)
     )
@@
   (symbol (lib_id "nets:-5V") (at 123.19 49.53 180)
     (in_bom yes) (on_board yes)
-    (property "Reference" "#PWR056" (id 0) (at 123.19 52.07 0)
+    (property "Reference" "#PWR064" (id 0) (at 123.19 52.07 0)
       (effects (font (size 1.27 1.27)) hide)
     )
@@
   (symbol (lib_id "mppcInterface-rescue:GND-power") (at 36.83 38.1 0)
     (in_bom yes) (on_board yes)
-    (property "Reference" "#PWR052" (id 0) (at 36.83 44.45 0)
+    (property "Reference" "#PWR060" (id 0) (at 36.83 44.45 0)
       (effects (font (size 1.27 1.27)) hide)
     )
@@
   (symbol (lib_id "nets:GND") (at 50.8 49.53 0)
     (in_bom yes) (on_board yes)
-    (property "Reference" "#PWR055" (id 0) (at 50.8 55.88 0)
+    (property "Reference" "#PWR063" (id 0) (at 50.8 55.88 0)
       (effects (font (size 1.27 1.27)) hide)
     )
@@
   (symbol (lib_id "nets:GND") (at 59.69 38.1 0)
     (in_bom yes) (on_board yes)
-    (property "Reference" "#PWR053" (id 0) (at 59.69 44.45 0)
+    (property "Reference" "#PWR061" (id 0) (at 59.69 44.45 0)
       (effects (font (size 1.27 1.27)) hide)
     )
@@
   (symbol (lib_id "nets:GND") (at 127 34.29 0)
     (in_bom yes) (on_board yes)
-    (property "Reference" "#PWR051" (id 0) (at 127 40.64 0)
+    (property "Reference" "#PWR059" (id 0) (at 127 40.64 0)
       (effects (font (size 1.27 1.27)) hide)
     )
@@
   (symbol (lib_id "passives:R-0402") (at 31.75 27.94 270)
     (in_bom yes) (on_board yes)
-    (property "Reference" "R6" (id 0) (at 31.75 22.733 90))
+    (property "Reference" "R10" (id 0) (at 31.75 22.733 90))
     (property "Value" "1K" (id 1) (at 31.75 25.0444 90))
     (property "Footprint" "passives:R-0402" (id 2) (at 31.496 28.956 90)
@@
   (symbol (lib_id "passives:R-0402") (at 55.88 48.26 90)
     (in_bom yes) (on_board yes)
-    (property "Reference" "R8" (id 0) (at 55.88 53.34 90))
+    (property "Reference" "R12" (id 0) (at 55.88 53.34 90))
     (property "Value" "49R9" (id 1) (at 55.88 50.8 90))
     (property "Footprint" "passives:R-0402" (id 2) (at 56.134 47.244 90)
@@
   (symbol (lib_id "passives:R-0402") (at 59.69 33.02 180)
     (in_bom yes) (on_board yes)
-    (property "Reference" "R7" (id 0) (at 58.42 33.02 0)
+    (property "Reference" "R11" (id 0) (at 58.42 33.02 0)
       (effects (font (size 1.27 1.27)) (justify left))
     )
@@
   (symbol (lib_id "passives:R-0402") (at 68.58 48.26 270)
     (in_bom yes) (on_board yes)
-    (property "Reference" "R9" (id 0) (at 68.58 53.34 90))
+    (property "Reference" "R13" (id 0) (at 68.58 53.34 90))
     (property "Value" "20K" (id 1) (at 68.58 50.8 90))
     (property "Footprint" "passives:R-0402" (id 2) (at 68.326 49.276 90)
@@
   (symbol (lib_id "passives:C-0402") (at 36.83 33.02 0)
     (in_bom yes) (on_board yes)
-    (property "Reference" "C27" (id 0) (at 34.29 31.75 0)
+    (property "Reference" "C32" (id 0) (at 34.29 31.75 0)
       (effects (font (size 1.27 1.27)) (justify right))
     )
-    (property "Value" "47n" (id 1) (at 34.29 34.29 0)
+    (property "Value" "0u1" (id 1) (at 34.29 34.29 0)
       (effects (font (size 1.27 1.27)) (justify right))
     )
@@
   (symbol (lib_id "passives:C-0402") (at 54.61 27.94 270)
     (in_bom yes) (on_board yes)
-    (property "Reference" "C24" (id 0) (at 54.61 21.5392 90))
+    (property "Reference" "C29" (id 0) (at 54.61 21.5392 90))
     (property "Value" "1u" (id 1) (at 54.61 23.8506 90))
     (property "Footprint" "passives:C-0402" (id 2) (at 50.8 28.9052 0)
@@
   (symbol (lib_id "passives:C-0402") (at 85.09 30.48 270)
     (in_bom yes) (on_board yes)
-    (property "Reference" "C26" (id 0) (at 85.09 24.0792 90))
+    (property "Reference" "C31" (id 0) (at 85.09 24.0792 90))
     (property "Value" "1u" (id 1) (at 85.09 26.3906 90))
     (property "Footprint" "passives:C-0402" (id 2) (at 81.28 31.4452 0)
@@
   (symbol (lib_id "passives:C-0402") (at 123.19 27.94 0)
     (in_bom yes) (on_board yes)
-    (property "Reference" "C25" (id 0) (at 126.111 26.7716 0)
+    (property "Reference" "C30" (id 0) (at 126.111 26.7716 0)
       (effects (font (size 1.27 1.27)) (justify left))
     )
@@
   (symbol (lib_id "passives:C-0402") (at 123.19 43.18 0)
     (in_bom yes) (on_board yes)
-    (property "Reference" "C28" (id 0) (at 126.111 42.0116 0)
+    (property "Reference" "C33" (id 0) (at 126.111 42.0116 0)
       (effects (font (size 1.27 1.27)) (justify left))
     )
@@
   (symbol (lib_id "U.FL:U.FL") (at 43.18 27.94 0) (mirror y)
     (in_bom yes) (on_board yes)
-    (property "Reference" "J1" (id 0) (at 44.958 21.8948 0))
+    (property "Reference" "J2" (id 0) (at 44.958 21.8948 0))
     (property "Value" "Conn_Coaxial" (id 1) (at 44.958 24.2062 0))
     (property "Footprint" "U.FL:U.FL" (id 2) (at 43.18 27.94 0)
@@
   (symbol (lib_id "OPA84X:OPA846") (at 68.58 30.48 0)
     (in_bom yes) (on_board yes)
-    (property "Reference" "U1" (id 0) (at 71.12 26.67 0)
-      (effects (font (size 1.27 1.27)) (justify left))
-    )
+    (property "Reference" "U2" (id 0) (at 71.12 26.67 0)
+      (effects (font (size 1.27 1.27)) (justify left))
+    )

Commit message: Updating gateware
Parts:
- renumbered C29 to C24, C30 to C25, C31 to C26, C32 to C27, C33 to C28, J2 to J1, R10 to R6, R11 to R7, R12 to R8, R13 to R9, U2 to U1
