File: pcb/mppcInterface.kicad_pcb (KiCad board)
At the start: 4 copper layers, 65 x 30 mm, 161 parts, among them J1 Conn_Coaxial, J2 Conn_Coaxial, J3 Conn_Coaxial, J4 Conn_Coaxial, J5 Conn_Coaxial, J6 Conn_Coaxial, J7 Conn_Coaxial, J8 Conn_Coaxial, J9 Raspberry_Pi_40P-Connector, Q1 BSS123L, U1 OPA846, U10 MIC5504-1.2YM5, U11 MAX1932, U12 DAC60508ZRTE, U13 MEA1D0505DC, U2 OPA846, U3 OPA846, U4 OPA846, U5 OPA846, U6 OPA846, U7 OPA846, U8 OPA846, U9 ICE40-LP384-SG32

Commit message: Updating gateware
Parts:
- removed C4: 1u, passives:C-0402
- removed D1, D2, D3: BL-HUB37A-AV-TRB, BL-HUB37A-AV-TRB:D-0402
- removed J9: Raspberry_Pi_40P-Connector, RaspberryPi:C35165
- removed TP10: GND, tooling:TestPoint_Pad_D1.0mm
- removed U9: ICE40-LP384-SG32, ICE40-LP384:ICE40-LP384-QFN32
- added D4: LL4148, LL4148:SOD-80, F.Cu at (43.4, -7.80)
- added TP11: 25, tooling:0.1in Pin, F.Cu at (16.5, 14.0)
- added TP12: 23, tooling:0.1in Pin, F.Cu at (11.4, 16.5)
- added TP13: 27, tooling:0.1in Pin, F.Cu at (16.5, 8.89)
- added TP14: 26, tooling:0.1in Pin, F.Cu at (16.5, 11.4)
- added TP15: 28, tooling:0.1in Pin, F.Cu at (16.5, 6.35)
- added TP16: 31, tooling:0.1in Pin, F.Cu at (16.5, -1.27)
- added TP17: 32, tooling:0.1in Pin, F.Cu at (16.5, -3.81)
- added TP18: 34, tooling:0.1in Pin, F.Cu at (16.5, -8.89)
- added TP19: 37, tooling:0.1in Pin, F.Cu at (14.0, -16.5)
- added TP20: CLK, tooling:0.1in Pin, F.Cu at (16.5, -11.4)
- added TP21: 36, tooling:0.1in Pin, F.Cu at (16.5, -14.0)
- added TP22: 43, tooling:0.1in Pin, F.Cu at (-1.27, -16.5)
- added TP23: 38, tooling:0.1in Pin, F.Cu at (11.4, -16.5)
- added TP24: 42, tooling:0.1in Pin, F.Cu at (1.27, -16.5)
- added TP25: 1V2, tooling:0.1in Pin, F.Cu at (16.5, 1.27)
- added TP26: 1V2, tooling:0.1in Pin, F.Cu at (16.5, 3.81)
- added TP27: 3V3, tooling:0.1in Pin, F.Cu at (14.0, 16.5)
- added TP28: 3V3, tooling:0.1in Pin, F.Cu at (8.89, 16.5)
- added TP29: DAC3, tooling:0.1in Pin, F.Cu at (-38.1, 33.0)
- added TP30: DAC2, tooling:0.1in Pin, F.Cu at (-40.6, 30.5)
- added TP31: DAC1, tooling:0.1in Pin, F.Cu at (-40.6, 27.9)
- added TP32: DAC0, tooling:0.1in Pin, F.Cu at (-40.6, 25.4)
- added TP33: DAC4, tooling:0.1in Pin, F.Cu at (-30.5, 33.0)
- added TP34: DAC5, tooling:0.1in Pin, F.Cu at (-27.9, 30.5)
- added TP35: DAC6, tooling:0.1in Pin, F.Cu at (-27.9, 27.9)
- added TP36: DAC7, tooling:0.1in Pin, F.Cu at (-27.9, 25.4)
- added TP37: RGB0, tooling:0.1in Pin, F.Cu at (8.89, -16.5)
- added TP38: RGB1, tooling:0.1in Pin, F.Cu at (6.35, -16.5)
- added TP39: RGB2, tooling:0.1in Pin, F.Cu at (3.81, -16.5)
- added TP40: 46, tooling:0.1in Pin, F.Cu at (-8.89, -16.5)
- added TP41: 47, tooling:0.1in Pin, F.Cu at (-11.4, -16.5)
- added TP42: 44, tooling:0.1in Pin, F.Cu at (-3.81, -16.5)
- added TP43: 48, tooling:0.1in Pin, F.Cu at (-14.0, -16.5)
- added TP44: 45, tooling:0.1in Pin, F.Cu at (-6.35, -16.5)
- added TP45: 02, tooling:0.1in Pin, F.Cu at (-16.5, -11.4)
- added TP46: 04, tooling:0.1in Pin, F.Cu at (-16.5, -6.35)
- added TP47: 03, tooling:0.1in Pin, F.Cu at (-16.5, -8.89)
- added TP48: ~{CS_{FPGA}}, tooling:0.1in Pin, F.Cu at (-6.35, 16.5)
- added TP49: SCLK, tooling:0.1in Pin, F.Cu at (-8.89, 16.5)
- added TP50: MOSI, tooling:0.1in Pin, F.Cu at (-3.81, 16.5)
- added TP51: MISO, tooling:0.1in Pin, F.Cu at (-11.4, 16.5)
- added TP52: 06, tooling:0.1in Pin, F.Cu at (-16.5, -1.27)
- added TP53: 09, tooling:0.1in Pin, F.Cu at (-16.5, 6.35)
- added TP54: 10, tooling:0.1in Pin, F.Cu at (-16.5, 8.89)
- added TP55: 11, tooling:0.1in Pin, F.Cu at (-16.5, 11.4)
- added TP56: 12, tooling:0.1in Pin, F.Cu at (-16.5, 14.0)
- added TP57: 21, tooling:0.1in Pin, F.Cu at (6.35, 16.5)
- added TP58: 13, tooling:0.1in Pin, F.Cu at (-14.0, 16.5)
- added TP59: 20, tooling:0.1in Pin, F.Cu at (3.81, 16.5)
- added TP60: 19, tooling:0.1in Pin, F.Cu at (1.27, 16.5)
- added TP61: 18, tooling:0.1in Pin, F.Cu at (-1.27, 16.5)
- added TP62: ~{FR}, tooling:0.1in Pin, F.Cu at (-16.5, 3.81)
- added TP63: FD, tooling:0.1in Pin, F.Cu at (-16.5, 1.27)
- added TP64: 1V2, tooling:0.1in Pin, F.Cu at (-16.5, -3.81)
- added TP65: 3V3, tooling:0.1in Pin, F.Cu at (-16.5, -14.0)
- added TP66: 3V3, tooling:0.1in Pin, F.Cu at (16.5, -6.35)
- added TP67: GND, tooling:0.1in Pin, F.Cu at (21.6, -1.27)
- added TP68: MISO, tooling:0.1in Pin, F.Cu at (-35.6, 20.3)
- added TP69: MOSI, tooling:0.1in Pin, F.Cu at (-33.0, 20.3)
- added TP70: SCLK, tooling:0.1in Pin, F.Cu at (-30.5, 20.3)
- added TP71: ~{CS_{DAC}}, tooling:0.1in Pin, F.Cu at (-27.9, 22.9)
- added TP72: ~{CS_{HV}}, tooling:0.1in Pin, F.Cu at (47.0, -3.81)
- added TP73: SCLK, tooling:0.1in Pin, F.Cu at (47.0, -6.35)
- added TP74: MOSI, tooling:0.1in Pin, F.Cu at (47.0, -8.89)
- added TP75: ~{CL}, tooling:0.1in Pin, F.Cu at (47.0, -11.4)
- added TP76: GND, tooling:0.1in Pin, F.Cu at (47.0, -1.27)
- added TP77: 3V3, tooling:0.1in Pin, F.Cu at (-38.1, 20.3)
- added TP78: 3V3, tooling:0.1in Pin, F.Cu at (-33.0, 33.0)
- added TP79: GND, tooling:0.1in Pin, F.Cu at (-35.6, 33.0)
- added TP80: 3V3, tooling:0.1in Pin, F.Cu at (57.1, -25.4)
- added TP81: GND, tooling:0.1in Pin, F.Cu at (47.0, 12.7)
- added TP82: HV, tooling:0.1in Pin, F.Cu at (47.0, 10.2)
- added U14: ICE40UP5K-SG48ITR50, ICE40-UP5K:ICE40-UP5K-SG48I, F.Cu at (0.00, 0.00)
- C2: value 1u -> 0u1
- C22, C23: footprint passives:C-0805 -> passives:C-0402
- C27, C32, C37, C42, C47, C52, C57, C62: value 47n -> 0u1
- H2, H3, H4: moved to F.Cu
- TP9: value HV -> 5V; footprint tooling:TestPoint_Pad_D1.0mm -> tooling:0.1in Pin
- moved C14 122.6 mm to (79.6, -60.9)
- moved C17 122.6 mm to (102.7, -63.6)
- moved C18 122.6 mm to (79.6, -62.7)
- moved C68 122.6 mm to (102.7, -60.0)
- moved FD3 122.6 mm to (91.2, -65.0)
- moved JP1 122.6 mm to (77.2, -55.2)
- moved L5 122.6 mm to (79.6, -59.1)
- moved L6 122.6 mm to (79.6, -64.5)
- moved L7 122.6 mm to (102.7, -61.8)
- moved U13 122.6 mm to (91.2, -61.8)
- moved C15 100.6 mm to (122.8, -10.8)
- moved C16 100.6 mm to (73.8, -9.40)
- moved C19 100.6 mm to (123.6, -12.7)
- moved C20 100.6 mm to (75.1, -8.90)
- moved C24 100.6 mm to (77.5, -7.90)
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Connections:
- C1 pad 2: +5V -> +3V3
- C2 pad 2: +5V -> +1V2
- C3 pad 2: +5V -> +1V2
- TP9 pad 1: HV -> +5V
- U10 pad 4: (no net) -> unconnected-(U10-NC-Pad4)
- U11 pad 12: ~CS_{HV} -> ~{CS_{HV}}
- U11 pad 3: (no net) -> ~{CL}
- U12 pad 1: (no net) -> unconnected-(U12-REF-Pad1)
- U12 pad 12: ~CS_{DAC} -> ~{CS_{DAC}}
- U12 pad 7: +5V -> +3V3
Routing:
- net GND: track 521.5 -> 247.9 mm, vias 66 -> 90
- net (no net): track 0.00 -> 135.5 mm, vias 0 -> 10
- net +5V: track 94.4 -> 3.40 mm, vias 8 -> 2
- net HV: track 77.1 -> 13.0 mm, vias 9 -> 8
- net -5V: track 94.2 -> 30.3 mm
- net +5V-A: track 84.7 -> 25.7 mm
- net +3V3: track 108.9 -> 143.6 mm, vias 6 -> 10
- net +1V2: track 31.3 -> 62.8 mm, vias 2 -> 4
- net GPIO18: track 30.6 -> 0.00 mm, vias 1 -> 0
- net ~CS_{DAC}: track 30.4 -> 0.00 mm, vias 1 -> 0
- net GPIO23: track 28.7 -> 0.00 mm, vias 1 -> 0
- net GPIO22: track 28.4 -> 0.00 mm, vias 1 -> 0
- net GPIO17: track 27.5 -> 0.00 mm, vias 2 -> 0
- net ~FPGA_{RST}: track 26.3 -> 0.00 mm, vias 1 -> 0
- net ~CS_{FPGA}: track 26.3 -> 0.00 mm, vias 3 -> 0
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- removed copper zone on In2.Cu, net +3V3
- removed copper zone on F.Cu, net +5V
- removed copper zone on In2.Cu, net +5V
- removed copper zone on In2.Cu, net +5V-A
- removed copper zone on In2.Cu, net -5V
- removed copper zone on In2.Cu, net /5V-BOOST
- removed copper zone on In1.Cu, net GND
- removed copper zone on In2.Cu, net GND
- removed copper zone on F.Cu, net HV
- removed copper zone on F.Cu, net Net-(D4-A)
- removed copper zone on F.Cu, net Net-(D4-K)
- removed copper zone on F.Cu, net Net-(U11-CS-)
Other:
- board size 65 x 30 mm -> 100 x 100 mm
- copper layers 4 -> 2
- board text added: "FPGA 1V2"
- board text removed: "GND"
