File: pcb/mppcInterface.kicad_sch (KiCad schematic)
At the start: 73 parts, among them J9 Raspberry_Pi_40P-Connector, Q1 BSS123L, U10 MIC5504-1.2YM5, U11 MAX1932, U12 DAC60508ZRTE, U13 MEA1D0505DC, U9 ICE40-LP384-SG32

Commit message: Updating gateware
Parts:
- removed C4: 1u, passives:C-0402, symbol passives:C-0402
- removed D1, D2, D3: BL-HUB37A-AV-TRB, BL-HUB37A-AV-TRB:D-0402, symbol BL-HUB37A-AV-TRB:BL-HUB37A-AV-TRB
- removed J9: Raspberry_Pi_40P-Connector, RaspberryPi:C35165, symbol RaspberryPi:Raspberry_Pi_40P-Connector
- removed TP10: GND, tooling:TestPoint_Pad_D1.0mm, symbol tooling:TestPoint_D1.0
- removed TP9: HV, tooling:TestPoint_Pad_D1.0mm, symbol tooling:TestPoint_D1.0
- removed U9: ICE40-LP384-SG32, ICE40-LP384:ICE40-LP384-QFN32, symbol ICE40-LP384:ICE40-LP384-SG32
- added TP11: 25, tooling:0.1in Pin, symbol tooling:TestPoint_TH-0.8
- added TP12: 23, tooling:0.1in Pin, symbol tooling:TestPoint_TH-0.8
- added TP13: 27, tooling:0.1in Pin, symbol tooling:TestPoint_TH-0.8
- added TP14: 26, tooling:0.1in Pin, symbol tooling:TestPoint_TH-0.8
- added TP15: 28, tooling:0.1in Pin, symbol tooling:TestPoint_TH-0.8
- added TP16: 31, tooling:0.1in Pin, symbol tooling:TestPoint_TH-0.8
- added TP17: 32, tooling:0.1in Pin, symbol tooling:TestPoint_TH-0.8
- added TP18: 34, tooling:0.1in Pin, symbol tooling:TestPoint_TH-0.8
- added TP19: 37, tooling:0.1in Pin, symbol tooling:TestPoint_TH-0.8
- added TP20: CLK, tooling:0.1in Pin, symbol tooling:TestPoint_TH-0.8
- added TP21: 36, tooling:0.1in Pin, symbol tooling:TestPoint_TH-0.8
- added TP22: 43, tooling:0.1in Pin, symbol tooling:TestPoint_TH-0.8
- added TP23: 38, tooling:0.1in Pin, symbol tooling:TestPoint_TH-0.8
- added TP24: 42, tooling:0.1in Pin, symbol tooling:TestPoint_TH-0.8
- added TP25, TP26, TP64: 1V2, tooling:0.1in Pin, symbol tooling:TestPoint_TH-0.8
- added TP27, TP28, TP65, TP66, TP77, TP78, TP80: 3V3, tooling:0.1in Pin, symbol tooling:TestPoint_TH-0.8
- added TP29: DAC3, tooling:0.1in Pin, symbol tooling:TestPoint_TH-0.8
- added TP30: DAC2, tooling:0.1in Pin, symbol tooling:TestPoint_TH-0.8
- added TP31: DAC1, tooling:0.1in Pin, symbol tooling:TestPoint_TH-0.8
- added TP32: DAC0, tooling:0.1in Pin, symbol tooling:TestPoint_TH-0.8
- added TP33: DAC4, tooling:0.1in Pin, symbol tooling:TestPoint_TH-0.8
- added TP34: DAC5, tooling:0.1in Pin, symbol tooling:TestPoint_TH-0.8
- added TP35: DAC6, tooling:0.1in Pin, symbol tooling:TestPoint_TH-0.8
- added TP36: DAC7, tooling:0.1in Pin, symbol tooling:TestPoint_TH-0.8
- added TP37: RGB0, tooling:0.1in Pin, symbol tooling:TestPoint_TH-0.8
- added TP38: RGB1, tooling:0.1in Pin, symbol tooling:TestPoint_TH-0.8
- added TP39: RGB2, tooling:0.1in Pin, symbol tooling:TestPoint_TH-0.8
- added TP40: 46, tooling:0.1in Pin, symbol tooling:TestPoint_TH-0.8
- added TP41: 47, tooling:0.1in Pin, symbol tooling:TestPoint_TH-0.8
- added TP42: 44, tooling:0.1in Pin, symbol tooling:TestPoint_TH-0.8
- added TP43: 48, tooling:0.1in Pin, symbol tooling:TestPoint_TH-0.8
- added TP44: 45, tooling:0.1in Pin, symbol tooling:TestPoint_TH-0.8
- added TP45: 02, tooling:0.1in Pin, symbol tooling:TestPoint_TH-0.8
- added TP46: 04, tooling:0.1in Pin, symbol tooling:TestPoint_TH-0.8
- added TP47: 03, tooling:0.1in Pin, symbol tooling:TestPoint_TH-0.8
- added TP48: ~{CS_{FPGA}}, tooling:0.1in Pin, symbol tooling:TestPoint_TH-0.8
- added TP49, TP70, TP73: SCLK, tooling:0.1in Pin, symbol tooling:TestPoint_TH-0.8
- added TP50, TP69, TP74: MOSI, tooling:0.1in Pin, symbol tooling:TestPoint_TH-0.8
- added TP51, TP68: MISO, tooling:0.1in Pin, symbol tooling:TestPoint_TH-0.8
- added TP52: 06, tooling:0.1in Pin, symbol tooling:TestPoint_TH-0.8
- added TP53: 09, tooling:0.1in Pin, symbol tooling:TestPoint_TH-0.8
- added TP54: 10, tooling:0.1in Pin, symbol tooling:TestPoint_TH-0.8
- added TP55: 11, tooling:0.1in Pin, symbol tooling:TestPoint_TH-0.8
- added TP56: 12, tooling:0.1in Pin, symbol tooling:TestPoint_TH-0.8
- added TP57: 21, tooling:0.1in Pin, symbol tooling:TestPoint_TH-0.8
- added TP58: 13, tooling:0.1in Pin, symbol tooling:TestPoint_TH-0.8
- added TP59: 20, tooling:0.1in Pin, symbol tooling:TestPoint_TH-0.8
- added TP60: 19, tooling:0.1in Pin, symbol tooling:TestPoint_TH-0.8
- added TP61: 18, tooling:0.1in Pin, symbol tooling:TestPoint_TH-0.8
- added TP62: ~{FR}, tooling:0.1in Pin, symbol tooling:TestPoint_TH-0.8
- added TP63: FD, tooling:0.1in Pin, symbol tooling:TestPoint_TH-0.8
- added TP67, TP76, TP79, TP81: GND, tooling:0.1in Pin, symbol tooling:TestPoint_TH-0.8
- added TP71: ~{CS_{DAC}}, tooling:0.1in Pin, symbol tooling:TestPoint_TH-0.8
- added TP72: ~{CS_{HV}}, tooling:0.1in Pin, symbol tooling:TestPoint_TH-0.8
- added TP75: ~{CL}, tooling:0.1in Pin, symbol tooling:TestPoint_TH-0.8
- added TP82: HV, tooling:0.1in Pin, symbol tooling:TestPoint_TH-0.8
- added TP9: 5V, tooling:0.1in Pin, symbol tooling:TestPoint_TH-0.8
- added U14: ICE40UP5K-SG48ITR50, ICE40-UP5K:ICE40-UP5K-SG48I, symbol ICE40-UP5K:ICE40UP5K-SG48ITR50
- C13: value 10u -> 4u7
- C2: value 1u -> 0u1
- C22, C23: footprint passives:C-0805 -> passives:C-0402; symbol passives:C-0805 -> passives:C-0402
Connections:
- net +1V2: now also C2.2, C3.2, TP25.1, TP26.1, TP64.1, U14.29 (VCCPLL), U14.30 (VCC), U14.5 (VCC)
- net +3V3: now also C1.2, U12.7 (VDD), TP27.1, TP28.1, TP65.1, TP66.1, TP77.1, TP78.1, TP80.1, U14.1 (VCCIO_2), U14.22 (SPI_VCCIO_1), U14.24 (VPP_2V5), U14.33 (VCCIO_0)
- net +5V: now also TP9.1; no longer C1.2, C2.2, C3.2, U12.7 (VDD)
- net CLK: now also TP20.1, U14.35 (IOT_46B_G0)
- net DAC0: now also TP32.1
- net DAC1: now also TP31.1
- net DAC2: now also TP30.1
- net DAC3: now also TP29.1
- net DAC4: now also TP33.1
- net DAC5: now also TP34.1
- net DAC6: now also TP35.1
- net DAC7: now also TP36.1
- net FPGA_{DONE}: now also TP63.1, U14.7 (CDONE)
- net GND: now also TP67.1, TP76.1, TP79.1, TP81.1, U14.EP (GND)
- net HV: now also TP82.1
- net MISO: now also TP51.1, TP68.1, U14.14 (IOB_32A_SPI_SO)
- net MOSI: now also TP50.1, TP69.1, TP74.1, U14.17 (IOB_33B_SPI_SI)
- net SCLK: now also TP49.1, TP70.1, TP73.1, U14.15 (IOB_34A_SPI_SCK)
- net ~CL renamed ~{CL}
- net ~{CL}: now also TP75.1
- net ~CS_{DAC} renamed ~{CS_{DAC}}
- net ~{CS_{DAC}}: now also TP71.1
- net ~CS_{HV} renamed ~{CS_{HV}}
- net ~{CS_{HV}}: now also TP72.1
- new net 02: TP45.1, U14.2 (IOB_6A)
- new net 03: TP47.1, U14.3 (IOB_9B)
- new net 04: TP46.1, U14.4 (IOB_8A)
- new net 06: TP52.1, U14.6 (IOB_13B)
- new net 09: TP53.1, U14.9 (IOB_16A)
- new net 10: TP54.1, U14.10 (IOB_18A)
- new net 11: TP55.1, U14.11 (IOB_20A)
- new net 12: TP56.1, U14.12 (IOB_22A)
- new net 13: TP58.1, U14.13 (IOB_24A)
- new net 18: TP61.1, U14.18 (IOB_31B)
- new net 19: TP60.1, U14.19 (IOB_29B)
- new net 20: TP59.1, U14.20 (IOB_25B_G3)
- new net 21: TP57.1, U14.21 (IOB_23B)
- new net 23: TP12.1, U14.23 (IOT_37A)
- new net 25: TP11.1, U14.25 (IOT_36B)
- new net 26: TP14.1, U14.26 (IOT_39A)
- new net 27: TP13.1, U14.27 (IOT_38B)
- new net 28: TP15.1, U14.28 (IOT_41A)
- new net 31: TP16.1, U14.31 (IOT_42B)
- new net 32: TP17.1, U14.32 (IOT_43A)
- new net 34: TP18.1, U14.34 (IOT_44B)
- new net 36: TP21.1, U14.36 (IOT_48B)
- new net 37: TP19.1, U14.37 (IOT_45A_G1)
- new net 38: TP23.1, U14.38 (IOT_50B)
- new net 42: TP24.1, U14.42 (IOT_51A)
- new net 43: TP22.1, U14.43 (IOT_49A)
- new net 44: TP42.1, U14.44 (IOB_3B_G6)
- new net 45: TP44.1, U14.45 (IOB_5B)
- new net 46: TP40.1, U14.46 (IOB_0A)
- new net 47: TP41.1, U14.47 (IOB_2A)
- new net 48: TP43.1, U14.48 (IOB_4A)
- new net RGB0: TP37.1, U14.39 (RGB0)
- new net RGB1: TP38.1, U14.40 (RGB1)
- new net RGB2: TP39.1, U14.41 (RGB2)
- new net ~{CS_{FPGA}}: TP48.1, U14.16 (IOB_35B_SPI_SS)
- new net ~{FPGA_{RST}}: TP62.1, U14.8 (~{CRESET_B})
- no-connect marks 5 -> 1
Other:
- note removed: "Raspberry PI"
- moved on the sheet: C10, C66, C67, C9
